Commit message: add d415 for ros1 real robot camera

File: Universal_Robots_ROS2_Description/urdf/ur.urdf.xacro (robot description, xacro)
@@ -11,4 +11,6 @@
    <!-- the default value should raise an error in case this was called without defining the type -->
    <xacro:arg name="ur_type" default="ur3e"/>
+   <!-- Peerajak to choose camera for sim robot or real robot-->
+   <xacro:property name="is_sim_robot" value="$(arg is_sim_robot)" />
    <!-- parameters -->
    <xacro:arg name="tf_prefix" default="" />
@@ -94,7 +96,16 @@
        <!--<origin xyz="0.0 0 0.0" rpy="0 -1.57 1.57"/>-->
    </xacro:rg2_gripper>
-   <xacro:sensor_r430 prefix="wrist_rgbd" parent="base_link" >
-       <origin xyz="-0.25 -0.3 0.2" rpy="0 ${pi/3} ${pi/2}"/>
-   </xacro:sensor_r430>
+   <!-- Peerajak Sim robot here -->
+   <xacro:if value="${is_sim_robot}">
+       <xacro:sensor_r430 prefix="wrist_rgbd" parent="base_link">
+        <origin xyz="-0.25 -0.3 0.2" rpy="0 ${pi/3} ${pi/2}"/>
+       </xacro:sensor_r430>
+   </xacro:if>
+   <!-- Peerajak Real robot here-->
+   <xacro:unless value="${is_sim_robot}">
+       <xacro:sensor_d415 prefix="D415" parent="base_link" >
+        <origin xyz="-0.25 -0.3 0.2" rpy="0 ${pi/3} ${pi/2}"/>
+       </xacro:sensor_d415>
+   </xacro:unless>
    <!--<xacro:sensor_r430 prefix="camera" parent="base_link" >
        <origin xyz="0.8 0.5 0.2" rpy="0 ${pi/6} ${pi}"/>

File: robotnik_sensors/robotnik_sensors/urdf/all_sensors.urdf.xacro (robot description, xacro)
@@ -79,4 +79,6 @@
   <!-- Intel Realsense D435 -->
   <xacro:include filename="$(find robotnik_sensors)/urdf/intel_d435.urdf.xacro" />
+  <!-- Peerajak add Intel Realsense D415-->
+  <xacro:include filename="$(find robotnik_sensors)/urdf/intel_d415.urdf.xacro" />
   <!-- Velodyne VLP16 -->
   <xacro:include filename="$(find robotnik_sensors)/urdf/velodyne_vlp16.urdf.xacro" />

Commit message: first roughtly successful whole system, but still the accuracy is not high

File: Universal_Robots_ROS2_Description/urdf/ur.urdf.xacro (robot description, xacro)
@@ -105,5 +105,5 @@
    <xacro:unless value="${is_sim_robot}">
        <xacro:sensor_d415 prefix="D415" parent="base_link" >
-        <origin xyz="-0.25 -0.3 0.2" rpy="0 ${pi/3} ${pi/2}"/>
+        <origin xyz="-0.415 -0.375 0.31" rpy="1.57 1.197 0"/>
        </xacro:sensor_d415>
    </xacro:unless>

Commit message: hand-camera coordination complete with different camera positioning

File: Universal_Robots_ROS2_Description/urdf/ur.urdf.xacro (robot description, xacro)
@@ -97,9 +97,14 @@
    </xacro:rg2_gripper>
    <!-- Peerajak Sim robot here -->
+   <!-- peerajak this is originalxacro:if value="${is_sim_robot}">
+       <xacro:sensor_r430 prefix="wrist_rgbd" parent="base_link">
+        <origin xyz="-0.25 -0.3 0.2" rpy="0 ${pi/3} ${pi/2}"/>
+       </xacro:sensor_r430>
+   </xacro:if -->
    <xacro:if value="${is_sim_robot}">
        <xacro:sensor_r430 prefix="wrist_rgbd" parent="base_link">
         <origin xyz="-0.25 -0.3 0.2" rpy="0 ${pi/3} ${pi/2}"/>
        </xacro:sensor_r430>
-   </xacro:if>
+   </xacro:if> <!-- peerajak this is testing value-->
    <!-- Peerajak Real robot here-->
    <xacro:unless value="${is_sim_robot}">

Commit message: Real robot left only accuracy

File: Universal_Robots_ROS2_Description/urdf/ur.urdf.xacro (robot description, xacro)
@@ -108,6 +108,7 @@
    </xacro:if> <!-- peerajak this is testing value-->
    <!-- Peerajak Real robot here-->
+   <!-- Peerajak Do not to this. Because this is the solution. It will mess with the answer-->
    <xacro:unless value="${is_sim_robot}">
-       <xacro:sensor_d415 prefix="D415" parent="base_link" >
+       <xacro:sensor_d415 prefix="sol_D415" parent="base_link" >
         <origin xyz="-0.415 -0.375 0.31" rpy="1.57 1.197 0"/>
        </xacro:sensor_d415>

File: rg2_gripper_description/urdf/rg2_gripper.urdf.xacro (robot description, xacro)
@@ -38,5 +38,5 @@
         </gazebo>
         <!-- Aruco Marker -->
-        <joint name="${prefix}_aruco_joint" type="fixed">
+        <!--joint name="${prefix}_aruco_joint" type="fixed">
             <origin xyz="0.065 0.0 0.025" rpy="0.0 0.0 0.0" />
             <parent link="${prefix}_base_link"/>
@@ -53,14 +53,7 @@
                 <geometry>
                     <mesh filename="package://rg2_gripper_description/meshes/arucomarker45mm.dae" scale="1.0 1.0 1.0"/>
-                    <!--<-box size="0.1 0.1 0.01" />-->
-                </geometry>
-            </visual>
-            <!--<collision>
-                <origin xyz="0.0 0 0" rpy="0 0 0" />
-                <geometry>
-                    <mesh filename="package://rg2_gripper_description/meshes/aruco_marker1.dae" scale="1.0 1.0 1.0"/>
-                </geometry>
-            </collision>-->
-        </link>
+                </geometry>
+            </visual>
+        </link-->
         <!--<xacro:macro name="mimic_joint_plugin_gazebo" params="parent_joint mimic_joint has_pid:=false multiplier:=1.0 offset:=0 sensitiveness:=0.0 max_effort:=1.0 robot_namespace:=''">
             <gazebo>
