Commit message: finetune movement and camera param on web

File: rg2_gripper_description/urdf/rg2_gripper.urdf.xacro (robot description, xacro)
@@ -38,5 +38,5 @@
         </gazebo>
         <!-- Aruco Marker -->
-        <!--joint name="${prefix}_aruco_joint" type="fixed">
+        <joint name="${prefix}_aruco_joint" type="fixed">
             <origin xyz="0.065 0.0 0.025" rpy="0.0 0.0 0.0" />
             <parent link="${prefix}_base_link"/>
@@ -55,5 +55,5 @@
                 </geometry>
             </visual>
-        </link-->
+        </link>
         <!--<xacro:macro name="mimic_joint_plugin_gazebo" params="parent_joint mimic_joint has_pid:=false multiplier:=1.0 offset:=0 sensitiveness:=0.0 max_effort:=1.0 robot_namespace:=''">
             <gazebo>
